File: main.kicad_sch (KiCad schematic)
At the start: 38 parts

Commit message: Schematic is basically feature complete
Parts:
- removed C?: 0u1, Capacitor_SMD:C_0402_1005Metric, symbol Device:C
- removed J?: SMA, Connector_Coaxial:SMA_Amphenol_132289_EdgeMount, symbol Connector:Conn_Coaxial
- removed L1: 100n, Inductor_SMD:L_0402_1005Metric, symbol Device:L
- removed Q?: AO3400A, Package_TO_SOT_SMD:SOT-23, symbol Transistor_FET:AO3400A
- removed Q?: AO3401A, Package_TO_SOT_SMD:SOT-23, symbol Transistor_FET:AO3401A
- removed R? (x2): 10k, Resistor_SMD:R_0402_1005Metric, symbol Device:R
- removed R?: 10, Resistor_SMD:R_0603_1608Metric, symbol Device:R
- removed R? (x2): 0, Resistor_SMD:R_0603_1608Metric, symbol Device:R
- removed R?: 100k, Resistor_SMD:R_0402_1005Metric, symbol Device:R
- removed TP? (x3): TestPoint_Probe, symbol Connector:TestPoint_Probe
- removed U?: MAX-M10S, RF_GPS:ublox_MAX, symbol RF_GPS:MAX-M10S
- added C? (x2): 22p, Capacitor_SMD:C_0402_1005Metric, symbol Device:C
- added C?: 10n, Capacitor_SMD:C_0402_1005Metric, symbol Device:C
- added C?: 1u, Capacitor_SMD:C_0402_1005Metric, symbol Device:C
- added D1, D2: D_TVS, Diode_SMD:D_0402_1005Metric_Pad0.77x0.64mm_HandSolder, symbol Device:D_TVS
- added D6: 5V6, symbol Device:D_Zener
- added D?: LED_BGKR, symbol Device:LED_BGKR
- added R? (x3): 1k, Resistor_SMD:R_0402_1005Metric, symbol Device:R
- added R? (x2): 10k, Resistor_SMD:R_0402_1005Metric, symbol Device:R
- added SW?: Reset, symbol Switch:SW_SPST
- added TP?: TestPoint_Probe, symbol Connector:TestPoint_Probe
- added Y1: 32768Hz, Crystal:Crystal_SMD_3215-2Pin_3.2x1.5mm, symbol Device:Crystal
- J11, J12, J13: renamed from J?; now left out of the parts list
- J14: renamed from J?; value Conn_01x02 -> Boot
- J6: renamed from J?; value USB_C_Receptacle_USB2.0_16P -> USB_C_Receptacle_16P
- gave numbers to parts that had none: 1
Connections:
- net USB_VBUS is gone; now on net +3V3: U4.20 (PA9)
- net +3V3: now also R?.2, R?.2
- net CPU_nRST: now also C?.1, SW?.1 (A)
- net GND: now also C?.1, C?.2, C?.2, C?.2, D1.1 (A1), D2.1 (A1), D6.2 (A), D?.3 (K), SW?.2 (B), TP?.1
- net I2C_SCL: now also R?.1
- net I2C_SDA: now also R?.1
- net USB_D+: now also D1.2 (A2)
- net USB_D-: now also D2.2 (A2)
- net VBus: now also C?.2, D6.1 (K)
- net Blue: now reaches U4.19 (PA8)
- net Blue: now also R?.2
- net at U4.2 (PC14): now also C?.1, Y1.1
- net Green: now reaches U4.25 (PA15(JTDI))
- net Green: now also R?.2
- net at U4.3 (PC15): now also C?.1, Y1.2
- net BOOT0: now reaches J14.2 (Pin_2), R?.1, U4.31 (BOOT0)
- net EXTINT: no longer names the net of U4.13 (PA7)
- net EXTINT: no longer U4.14 (PB0)
- net GPIO0: no longer names the net of U4.11 (PA5)
- net GPIO1 renamed Alert
- new net: D?.1 (BA), R?.1
- new net: D?.2 (GA), R?.1
- new net: D?.4 (RA), R?.1
- new net Red: R?.2, U4.14 (PB0)
- no-connect marks 6 -> 3
Other:
- note added: "USB_VBUS"
- note removed: "Open for 3.3V"
- note removed: "TODO - Two pins left for LEDs!"
- note removed: "TODO - add prot circuit?"
- note removed: "TODO - not needed?"
- note removed: "TODO - protection."
- note removed: "TODO - reset filter & switch"
- moved on the sheet: C?, J11, J12, J13, J14, J6, R?, U4
