File: gpsref.kicad_sch (KiCad schematic)
At the start: 0 parts

Commit message: Schematic is basically feature complete
Other:
- sheet Main renamed CPU
- added sheet GPS (gps.kicad_sch)
Changed lines of the file:
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@@
 	(paper "A4")
 	(sheet
-		(at 41.91 74.93)
-		(size 40.64 17.78)
-		(exclude_from_sim no)
-		(in_bom yes)
-		(on_board yes)
-		(dnp no)
-		(fields_autoplaced yes)
+		(at 129.54 76.2)
+		(size 25.4 12.7)
+		(exclude_from_sim no)
+		(in_bom yes)
+		(on_board yes)
+		(dnp no)
 		(stroke
 			(width 0.1524)
@@
 		)
 		(property "Sheetname" "Clocking"
-			(at 41.91 74.2184 0)
-			(effects
-				(font
-					(size 1.27 1.27)
-				)
-				(justify left bottom)
+			(at 142.24 82.6004 0)
+			(effects
+				(font
+					(size 2.54 2.54)
+					(thickness 0.508)
+					(bold yes)
+				)
 			)
 		)
 		(property "Sheetfile" "clocking.kicad_sch"
-			(at 41.91 93.2946 0)
+			(at 129.54 89.4846 0)
 			(effects
 				(font
@@
 	)
 	(sheet
-		(at 146.05 34.29)
-		(size 36.83 20.32)
-		(exclude_from_sim no)
-		(in_bom yes)
-		(on_board yes)
-		(dnp no)
-		(fields_autoplaced yes)
+		(at 160.02 76.2)
+		(size 25.4 12.7)
+		(exclude_from_sim no)
+		(in_bom yes)
+		(on_board yes)
+		(dnp no)
 		(stroke
 			(width 0.1524)
@@
 		)
 		(property "Sheetname" "Outputs"
-			(at 146.05 33.5784 0)
-			(effects
-				(font
-					(size 1.27 1.27)
-				)
-				(justify left bottom)
+			(at 172.974 82.6004 0)
+			(effects
+				(font
+					(size 2.54 2.54)
+					(thickness 0.508)
+					(bold yes)
+				)
 			)
 		)
 		(property "Sheetfile" "output.kicad_sch"
-			(at 146.05 55.1946 0)
+			(at 160.02 89.4846 0)
 			(effects
 				(font
@@
 	)
 	(sheet
-		(at 43.18 40.64)
-		(size 33.02 17.78)
-		(exclude_from_sim no)
-		(in_bom yes)
-		(on_board yes)
-		(dnp no)
-		(fields_autoplaced yes)
+		(at 99.06 76.2)
+		(size 25.4 12.7)
+		(exclude_from_sim no)
+		(in_bom yes)
+		(on_board yes)
+		(dnp no)
+		(stroke
+			(width 0.1524)
+			(type solid)
+		)
+		(fill
+			(color 0 0 0 0.0000)
+		)
+		(property "Sheetname" "GPS"
+			(at 112.014 82.8544 0)
+			(effects
+				(font
+					(size 2.54 2.54)
+					(thickness 0.508)
+					(bold yes)
+				)
+			)
+		)
+		(property "Sheetfile" "gps.kicad_sch"
+			(at 99.06 89.4846 0)
+			(effects
+				(font
+					(size 1.27 1.27)
+				)
+				(justify left top)
+			)
+		)
+		(instances
+			(project "gpsref"
+				(path "/3160ff17-81c2-4674-af97-e8d9acaf6b65"
+					(page "1")
+				)
+			)
+		)
+	)
+	(sheet
+		(at 144.78 96.52)
+		(size 25.4 12.7)
+		(exclude_from_sim no)
+		(in_bom yes)
+		(on_board yes)
+		(dnp no)
 		(stroke
 			(width 0.1524)
@@
 		)
 		(property "Sheetname" "Power"
-			(at 43.18 39.9284 0)
-			(effects
-				(font
-					(size 1.27 1.27)
-				)
-				(justify left bottom)
+			(at 157.48 102.9204 0)
+			(effects
+				(font
+					(size 2.54 2.54)
+					(thickness 0.508)
+					(bold yes)
+				)
 			)
 		)
 		(property "Sheetfile" "power.kicad_sch"
-			(at 43.18 59.0046 0)
+			(at 144.78 110.0586 0)
+			(effects
+				(font
+					(size 1.27 1.27)
+				)
+				(justify left top)
+			)
+		)
+		(instances
+			(project "gpsref"
+				(path "/3160ff17-81c2-4674-af97-e8d9acaf6b65"
+					(page "5")
+				)
+			)
+		)
+	)
+	(sheet
+		(at 114.3 96.52)
+		(size 25.4 12.7)
+		(exclude_from_sim no)
+		(in_bom yes)
+		(on_board yes)
+		(dnp no)
+		(stroke
+			(width 0.1524)
+			(type solid)
+		)
+		(fill
+			(color 0 0 0 0.0000)
+		)
+		(property "Sheetname" "CPU"
+			(at 126.746 103.4284 0)
+			(effects
+				(font
+					(size 2.54 2.54)
+					(thickness 0.508)
+					(bold yes)
+				)
+			)
+		)
+		(property "Sheetfile" "main.kicad_sch"
+			(at 114.3 109.8046 0)
 			(effects
 				(font
@@
 				)
 			)
-		)
-	)
-	(sheet
-		(at 97.79 39.37)
-		(size 33.02 15.24)
-		(exclude_from_sim no)
-		(in_bom yes)
-		(on_board yes)
-		(dnp no)
-		(fields_autoplaced yes)
-		(stroke
-			(width 0.1524)
-			(type solid)
-		)
-		(fill
-			(color 0 0 0 0.0000)
-		)
-		(property "Sheetname" "Main"
-			(at 97.79 38.6584 0)
-			(effects
-				(font
-					(size 1.27 1.27)
-				)
-				(justify left bottom)
-			)
-		)
-		(property "Sheetfile" "main.kicad_sch"
-			(at 97.79 55.1946 0)
-			(effects
-				(font
-					(size 1.27 1.27)
-				)
-				(justify left top)
-			)
-		)
-		(instances
-			(project "gpsref"
-				(path "/3160ff17-81c2-4674-af97-e8d9acaf6b65"
-					(page "1")
-				)
-			)

Commit message: Sorting out the part placement....
Other:
- sheet CPU: file main.kicad_sch -> cpu.kicad_sch
Changed lines of the file:
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@@
 			)
 		)
-		(property "Sheetfile" "main.kicad_sch"
+		(property "Sheetfile" "cpu.kicad_sch"
 			(at 114.3 109.8046 0)
 			(effects
