File: gpsref.kicad_pcb (KiCad board)
At the start: 4 copper layers, 77.4 x 47.8 mm, 183 parts, among them J1 SMA, J11 Debug, J12 GPS_Snoop, J13 I2C_Snoop, J2 SMA, J3 SMA, J4 SMA, J5 U.Fl, J6 SMA, J7 USB_C_Receptacle_16P, Q1 AO3400A, Q2 AO3401A, T1 MABA-007159-000000, T2 MABA-007159-000000, U1 MAX-M10S, U12 74LVC1G125, U13 74CB3Q3306, U15 74LVC1G07, U2 TG5032CGN, U3 LMK05318BRGZR, U31 TMP117xxDRV, U4 STM32H503KBUx, U5 TPS82084SIL, U6 TPS82084SIL, U7 TPS7A8801RTJR, U9 TPS7A8801RTJR, Y1 32768Hz

Commit message: Redo the secondary reference termination.
Parts:
- removed C54: 0u1, Capacitor_SMD:C_0402_1005Metric
- R33: value 100 -> 200
- R35: renamed from R31; value 200 -> 0
- moved R33 36.9 mm to (153.6, 100.9), turned to 90 degrees
- moved TP7 9.10 mm to (132.2, 119.7)
- moved R35 3.33 mm to (152.8, 103.2), turned to 0 degrees
- moved R34 1.60 mm to (155.2, 100.9)
- moved L34 0.75 mm to (149.2, 102.6)
- renumbered R34 to R31, R35 to R34
Connections:
- C41 pad 1: CGEN_3V3 -> /Clocking/VDD_DIG
- R34 pad 1: GND -> Net-(R34-Pad1)
- R35 pad 1: /Clocking/SecRefLo -> GND
- R35 pad 2: /Clocking/VDD_DIG -> Net-(R34-Pad1)
- U31 pad 4: CGEN_3V3 -> /Clocking/VDD_DIG
- U31 pad 5: CGEN_3V3 -> /Clocking/VDD_DIG
Routing:
- net /Clocking/SecRefLo: track 52.2 -> 3.16 mm, vias 2 -> 0
- net SecRef: track 3.72 -> 51.6 mm, vias 0 -> 2
- net GND: track 189.9 -> 214.2 mm, vias 303 -> 300
- net CGEN_3V3: track 98.0 -> 84.6 mm, vias 9 -> 7
- net /Clocking/VDD_DIG: track 15.6 -> 21.3 mm, vias 2 -> 3
- net OUT4: track 46.9 -> 43.9 mm
- net Net-(R34-Pad1): track 0.00 -> 1.84 mm
- net EN_OUT4: track 35.1 -> 36.6 mm
- net +3V3: track 197.2 -> 197.3 mm, vias 14 -> 13
