File: cpu.kicad_sch (KiCad schematic)
At the start: 38 parts, among them J10 Skedd, J11 I2C_Snoop, J12 GPS_Snoop, J13 Boot, J7 USB_C_Receptacle_16P, U4 STM32H503KBUx, Y1 32768Hz

Commit message: Schematic updates for revision mostly done.
Parts:
- removed C41: 0u1, Capacitor_SMD:C_0402_1005Metric, symbol Device:C
- removed C44, C45: 22p, Capacitor_SMD:C_0402_1005Metric, symbol Device:C
- removed J10: Skedd, Parts:Skedd6, symbol Connector_Generic:Conn_02x03_Odd_Even
- removed J11: I2C_Snoop, Parts:PinHeader_1x04_P2.54mm_Vertical, symbol Connector:Conn_01x04_Pin
- removed J12: GPS_Snoop, Parts:PinHeader_1x03_P2.54mm_Vertical, symbol Connector:Conn_01x03_Pin
- removed R1, R2, R3, R4, R48, R49: 100, Resistor_SMD:R_0402_1005Metric, symbol Device:R
- removed R6: 10k, Resistor_SMD:R_0402_1005Metric, symbol Device:R
- removed Y1: 32768Hz, Crystal:Crystal_SMD_3215-2Pin_3.2x1.5mm, symbol Device:Crystal
- added C43: 10u, Capacitor_SMD:C_0402_1005Metric, symbol Device:C
- added L41: 220, Inductor_SMD:L_0603_1608Metric, symbol Parts:L_Ferrite_Power
- R50: renamed from R7; value 100 -> 100k; LCSC C25076 -> (none)
- renumbered C42 to C41, C43 to C42, C47 to C44, C48 to C45, C50 to C47, C49 to C48, D9 to D2, D10 to D3, D11 to D41, D12 to D42, R5 to R48, R8 to R49
Connections:
- net STATUS1 is gone; now on net GND: U4.12 (PA6)
- net dRX is gone; now on net dTX: J13.3 (Pin_3), R49.1
- net +3V3: now also L41.1; no longer C44.1, C45.1, D2.3 (A), U4.1 (VDD), U4.17 (VDD), U4.20 (PA9), U4.5 (VDDA)
- net DBG_TX: now also R49.2
- net GND: now also C43.2; no longer U4.11 (PA5), U4.13 (PA7)
- net DBG_RX: no longer names the net of U4.25 (PA15(JTDI))
- net DBG_RX: no longer R49.2
- net EN_OUT3: no longer names the net of U4.32 (PB8)
- net EN_OUT4: no longer names the net of U4.27 (PB4(NJTRST))
- net EN_REF2: no longer names the net of U4.28 (PB5)
- net SWCLK: no longer names the net of U4.24 (PA14(JTCK)
- net SWDIO: no longer names the net of U4.23 (PA13(JTMS)
- net X32In: no longer names the net of U4.2 (PC14)
- net X32Out: no longer names the net of U4.3 (PC15)
- new net FDEC: U4.13 (PA7)
- new net FINC: U4.11 (PA5)
- new net LED_PWR: D2.3 (A)
- new net VCPU: C43.1, C44.1, C45.1, L41.2, U4.1 (VDD), U4.17 (VDD), U4.20 (PA9), U4.5 (VDDA)
- no-connect marks 2 -> 10
Other:
- note added: "EN_OUT3"
- note added: "EN_OUT4"
- note added: "EN_REF2"
- moved on the sheet: C44, C45, C47, C48, J13, R48, R49, R50

Commit message: Use impedance matching baluns.
Connections:
- net LED_PWR is gone; now on net +3V3: D2.3 (A)
- net +3V3: no longer R46.2, R47.2
- net VCPU: now also R46.2, R47.2
