File: end-out.kicad_pcb (KiCad board)
At the start: 2 copper layers, 49.8 x 20 mm, 4 parts

Commit message: Add bias resistors to comparators.
Routing:
- net GND: vias 3 -> 4
- added copper zone on F.Cu, net GND
- removed copper zone on B.Cu, net GND
Other:
- outline, holes or cut-outs redrawn
- board text added: "1+"
- board text added: "1-"
- board text removed: "1"

Commit message: Copper fill on both sides of end-out also.
Routing:
- added copper zone on B.Cu, net GND
Changed lines of the file:
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@@
 		(net 1)
 		(net_name "GND")
-		(layer "F.Cu")
+		(layers "F.Cu" "B.Cu")
 		(name "Back")
 		(hatch edge 0.5)
-		(connect_pads
+		(connect_pads yes
 			(clearance 0.2)
 		)
