File: output-diff-sma.kicad_sch (KiCad schematic)
At the start: 6 parts

Commit message: FPGA in, layout mostly updated.
Parts:
- renumbered C30 to C11, C31 to C12
Changed lines of the file:
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@@
 		(in_pos_files yes)
 		(dnp no)
-		(property "Reference" "C30"
+		(property "Reference" "C11"
 			(at 65.786 61.976 90)
 			(show_name no)
@@
 			(project "gpsfreak"
 				(path "/3160ff17-81c2-4674-af97-e8d9acaf6b65/64bdf83b-4762-4d14-abd1-564acb81cb91"
-					(reference "C30")
+					(reference "C11")
 					(unit 1)
 				)
@@
 		(in_pos_files yes)
 		(dnp no)
-		(property "Reference" "C31"
+		(property "Reference" "C12"
 			(at 65.786 67.056 90)
 			(show_name no)
@@
 			(project "gpsfreak"
 				(path "/3160ff17-81c2-4674-af97-e8d9acaf6b65/64bdf83b-4762-4d14-abd1-564acb81cb91"
-					(reference "C31")
-					(unit 1)
-				)
+					(reference "C12")
+					(unit 1)
+				)

Commit message: Layout down
Parts:
- C11, C12: Stock (none) -> Basic
- D31, D32: Stock (none) -> N/A
- JN1, JP1: Stock (none) -> AliX
Changed lines of the file:
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@@
+			)
+		)
+		(property "Stock" "Basic"
+			(at 64.77 62.23 90)
+			(hide yes)
+			(show_name no)
+			(do_not_autoplace no)
+			(effects
+				(font
+					(size 1.27 1.27)
+				)
 			)
 		)
@@
 			)
 		)
+		(property "Stock" "N/A"
+			(at 54.61 71.12 90)
+			(hide yes)
+			(show_name no)
+			(do_not_autoplace no)
+			(effects
+				(font
+					(size 1.27 1.27)
+				)
+			)
+		)
 		(pin "2"
 		)
@@
 			)
 		)
+		(property "Stock" "AliX"
+			(at 87.63 62.23 0)
+			(hide yes)
+			(show_name no)
+			(do_not_autoplace no)
+			(effects
+				(font
+					(size 1.27 1.27)
+				)
+			)
+		)
 		(pin "2"
 		)
@@
 			)
 		)
+		(property "Stock" "N/A"
+			(at 54.61 58.42 90)
+			(hide yes)
+			(show_name no)
+			(do_not_autoplace no)
+			(effects
+				(font
+					(size 1.27 1.27)
+				)
+			)
+		)
 		(pin "2"
 		)
@@
 			)
 		)
+		(property "Stock" "AliX"
+			(at 78.74 67.31 0)
+			(hide yes)
+			(show_name no)
+			(do_not_autoplace no)
+			(effects
+				(font
+					(size 1.27 1.27)
+				)
+			)
+		)
 		(pin "2"
 		)
@@
 			(at 64.77 67.31 90)
 			(hide yes)
+			(show_name no)
+			(do_not_autoplace no)
+			(effects
+				(font
+					(size 1.27 1.27)
+				)
+			)
+		)
+		(property "Stock" "Basic"
+			(at 64.77 67.31 90)
+			(hide yes)
