File: output-passive.kicad_sch (KiCad schematic)
At the start: 16 parts, among them J4 SMA, U41 TS5A63157DBV

Commit message: Layout down
Parts:
- C4, C44, C45, C5, R48: Stock (none) -> Basic
- C43: LCSC (none) -> C32949; Stock (none) -> Basic
- D41: Stock (none) -> N/A
- D42: LCSC (none) -> C191023; Stock (none) -> Basic
- J4: Stock (none) -> AliX
- R41, R42, R43: LCSC (none) -> C25744; Stock (none) -> Basic
- R44: LCSC (none) -> C11702; Stock (none) -> Basic
- R45: LCSC (none) -> C25076; Stock (none) -> Basic
- R47: value 39 -> 33; LCSC (none) -> C25105; Stock (none) -> Basic
- U41: footprint Parts:SOT-353_SC-70-6 -> Parts:SOT-363_SC-70-6; LCSC (none) -> C133575; Stock (none) -> ORDER
Other:
- moved on the sheet: C44, D42, U41B

Commit message: Tidy up.
Parts:
- D42: value 1N5819WS -> RB751S-40; footprint Diode_SMD:D_SOD-323 -> Diode_SMD:D_SOD-523; LCSC C191023 -> C7502700; Stock Basic -> Prom
- renumbered C4 to C41, C5 to C42
Changed lines of the file:
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@@
 		(in_pos_files yes)
 		(dnp no)
-		(property "Reference" "C5"
+		(property "Reference" "C42"
 			(at 97.79 57.15 0)
 			(show_name no)
@@
 			(project "gpsfreak"
 				(path "/3160ff17-81c2-4674-af97-e8d9acaf6b65/8de00818-124c-4cc8-9910-e794140dfeb1"
-					(reference "C5")
+					(reference "C42")
 					(unit 1)
 				)
@@
 			)
 		)
-		(property "Value" "1N5819WS"
+		(property "Value" "RB751S-40"
 			(at 125.73 22.86 0)
 			(show_name no)
@@
 			)
 		)
-		(property "Footprint" "Diode_SMD:D_SOD-323"
+		(property "Footprint" "Diode_SMD:D_SOD-523"
 			(at 125.73 20.955 0)
 			(hide yes)
@@
 			)
 		)
-		(property "Datasheet" "https://datasheet.lcsc.com/lcsc/2204281430_Guangdong-Hottech-1N5819WS_C191023.pdf"
+		(property "Datasheet" ""
 			(at 125.73 25.4 0)
 			(hide yes)
@@
 			)
 		)
-		(property "Stock" "Basic"
+		(property "Stock" "Prom"
 			(at 125.73 25.4 0)
 			(hide yes)
@@
 			)
 		)
-		(property "LCSC" "C191023"
+		(property "LCSC" "C7502700"
 			(at 125.73 25.4 0)
 			(hide yes)
@@
 		(in_pos_files yes)
 		(dnp no)
-		(property "Reference" "C4"
+		(property "Reference" "C41"
 			(at 107.95 39.37 0)
 			(show_name no)
@@
 			(project "gpsfreak"
 				(path "/3160ff17-81c2-4674-af97-e8d9acaf6b65/8de00818-124c-4cc8-9910-e794140dfeb1"
-					(reference "C4")
+					(reference "C41")
 					(unit 1)
 				)

Commit message: Ordered.
Parts:
- U9: renamed from U41; now left out of the parts list
- renumbered R47 to R46, R48 to R47
Changed lines of the file:
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@@
 	(generator_version "10.0")
 	(paper "A4")
-	(text_box "Switch can be powered up via its protection diodes."
+	(text_box "Switch can be powered via its protection diodes."
 		(exclude_from_sim no)
 		(at 115.57 29.21 0)
@@
 		(in_pos_files yes)
 		(dnp no)
-		(property "Reference" "R47"
-			(at 128.27 71.882 90)
+		(property "Reference" "R46"
+			(at 128.27 67.818 90)
 			(show_name no)
 			(do_not_autoplace no)
@@
 			(project "gpsfreak"
 				(path "/3160ff17-81c2-4674-af97-e8d9acaf6b65/8de00818-124c-4cc8-9910-e794140dfeb1"
-					(reference "R47")
+					(reference "R46")
 					(unit 1)
 				)
@@
 		(body_style 1)
 		(exclude_from_sim no)
-		(in_bom yes)
+		(in_bom no)
 		(on_board yes)
 		(in_pos_files yes)
 		(dnp no)
-		(property "Reference" "U41"
+		(property "Reference" "U9"
 			(at 116.713 66.675 0)
 			(show_name no)
@@
 			(project "gpsfreak"
 				(path "/3160ff17-81c2-4674-af97-e8d9acaf6b65/8de00818-124c-4cc8-9910-e794140dfeb1"
-					(reference "U41")
+					(reference "U9")
 					(unit 1)
 				)
@@
 		(in_pos_files yes)
 		(dnp no)
-		(property "Reference" "R48"
+		(property "Reference" "R47"
 			(at 113.538 82.55 90)
 			(show_name no)
@@
 			(project "gpsfreak"
 				(path "/3160ff17-81c2-4674-af97-e8d9acaf6b65/8de00818-124c-4cc8-9910-e794140dfeb1"
-					(reference "R48")
+					(reference "R47")
 					(unit 1)
 				)
@@
 		(body_style 1)
 		(exclude_from_sim no)
-		(in_bom yes)
+		(in_bom no)
 		(on_board yes)
 		(in_pos_files yes)
 		(dnp no)
-		(property "Reference" "U41"
+		(property "Reference" "U9"
 			(at 147.193 37.973 0)
 			(show_name no)
@@
 			(project "gpsfreak"
 				(path "/3160ff17-81c2-4674-af97-e8d9acaf6b65/8de00818-124c-4cc8-9910-e794140dfeb1"
-					(reference "U41")
+					(reference "U9")
 					(unit 2)
 				)
