File: fpga.kicad_sch (KiCad schematic)
At the start: 24 parts, among them J8 Conn_01x06, SW1 SW_Push, U8 LCMXO2-640HC-4SG48C

Commit message: Tidy up.
Parts:
- added R11: 5k1, Resistor_SMD:R_0402_1005Metric, symbol Device:R
- U8: footprint Package_DFN_QFN:QFN-48-1EP_7x7mm_P0.5mm_EP5.45x5.45mm -> Parts:QFN-48-1EP_7x7mm_P0.5mm_EP5.45x5.45mm; LCSC (none) -> C1521838; now left out of the parts list
- renumbered C6 to C84
Connections:
- net ClkIO+: now also U8.18 (B6C); no longer U8.17 (B6B)
- net ClkIO-: now also U8.19 (B6D); no longer U8.18 (B6C)
- net ClkOEN: now also U8.11 (L6A); no longer U8.15 (B4B)
- net GPS_nRSTF: now also R87.2
- net VFPGA: now also R11.1
- net at R61.1, U8.26 (R7D): no longer R87.2
- net at U8.38 (T11C): now also R11.2
- no-connect marks 1 -> 18
Other:
- moved on the sheet: C81, C82, C83, C84, C85, C86, C87, C88, L81, R61, R62, R80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

Commit message: Ordered.
Parts:
- U8: now in the parts list
Changed lines of the file:
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@@
 		(body_style 1)
 		(exclude_from_sim no)
-		(in_bom no)
+		(in_bom yes)
 		(on_board yes)
 		(in_pos_files yes)

Commit message: Adjustments.  Silk screen clearance.
Parts:
- added R65: 100, Resistor_SMD:R_0402_1005Metric, symbol Device:R
Connections:
- net ClkIn+: now also R65.1
- net ClkIn-: now also R65.2
Changed lines of the file:
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@@
+	)
+	(junction
+		(at 156.21 80.01)
+		(diameter 0)
+		(color 0 0 0 0)
 	)
 	(junction
@@
 		(color 0 0 0 0)
 	)
+	(junction
+		(at 156.21 87.63)
+		(diameter 0)
+		(color 0 0 0 0)
+	)
 	(no_connect
 		(at 111.76 95.25)
@@
 	(wire
 		(pts
+			(xy 156.21 87.63) (xy 161.29 87.63)
+		)
+		(stroke
+			(width 0)
+			(type default)
+		)
+	)
+	(wire
+		(pts
 			(xy 161.29 63.5) (xy 163.83 63.5)
 		)
@@
 	(wire
 		(pts
+			(xy 153.67 82.55) (xy 153.67 80.01)
+		)
+		(stroke
+			(width 0)
+			(type default)
+		)
+	)
+	(wire
+		(pts
+			(xy 156.21 87.63) (xy 153.67 87.63)
+		)
+		(stroke
+			(width 0)
+			(type default)
+		)
+	)
+	(wire
+		(pts
 			(xy 152.4 102.87) (xy 153.67 102.87)
 		)
@@
 	(wire
 		(pts
+			(xy 156.21 80.01) (xy 161.29 80.01)
+		)
+		(stroke
+			(width 0)
+			(type default)
+		)
+	)
+	(wire
+		(pts
 			(xy 118.11 124.46) (xy 118.11 116.84)
 		)
@@
 	(wire
 		(pts
-			(xy 152.4 82.55) (xy 158.75 82.55)
+			(xy 152.4 82.55) (xy 153.67 82.55)
+		)
+		(stroke
+			(width 0)
+			(type default)
+		)
+	)
+	(wire
+		(pts
+			(xy 153.67 80.01) (xy 156.21 80.01)
 		)
 		(stroke
@@
 	(wire
 		(pts
-			(xy 152.4 85.09) (xy 158.75 85.09)
+			(xy 152.4 85.09) (xy 153.67 85.09)
 		)
 		(stroke
@@
 		(pts
 			(xy 146.05 53.34) (xy 144.78 53.34)
+		)
+		(stroke
+			(width 0)
+			(type default)
+		)
+	)
+	(wire
+		(pts
+			(xy 153.67 87.63) (xy 153.67 85.09)
 		)
 		(stroke
@@
 		(shape input)
 		(at 130.81 62.23 90)
-		(fields_autoplaced yes)
 		(effects
 			(font
@@
 		)
 		(property "Intersheetrefs" "${INTERSHEET_REFS}"
-			(at 130.81 51.6853 90)
+			(at 130.81 53.4633 90)
 			(show_name no)
 			(do_not_autoplace no)
@@
 		(shape bidirectional)
 		(at 133.35 62.23 90)
-		(fields_autoplaced yes)
 		(effects
 			(font
@@
 		)
 		(property "Intersheetrefs" "${INTERSHEET_REFS}"
-			(at 133.35 50.5135 90)
+			(at 133.35 52.2915 90)
 			(show_name no)
 			(do_not_autoplace no)
@@
 	)
 	(global_label "GPS_nRST"
-		(shape input)
+		(shape output)
 		(at 107.95 82.55 180)
 		(effects
@@
 	(hierarchical_label "ClkIn-"
 		(shape input)
-		(at 158.75 85.09 0)
+		(at 161.29 87.63 0)
 		(effects
 			(font
@@
 	(hierarchical_label "ClkIn+"
 		(shape input)
-		(at 158.75 82.55 0)
+		(at 161.29 80.01 0)
 		(effects
 			(font
@@
 		)
 		(property "Value" "LCMXO2-640HC-4SG48C"
-			(at 132.334 80.01 0)
+			(at 132.08 101.854 0)
 			(show_name no)
 			(do_not_autoplace no)
@@
 					(unit 1)
 				)
+			)
+		)
+	)
+	(symbol
+		(lib_id "Device:R")
+		(at 156.21 83.82 0)
+		(unit 1)
+		(body_style 1)
+		(exclude_from_sim no)
+		(in_bom yes)
+		(on_board yes)
+		(in_pos_files yes)
+		(dnp no)
+		(property "Reference" "R65"
+			(at 157.734 83.82 90)
+			(show_name no)
+			(do_not_autoplace no)
+			(effects
+				(font
+					(size 1.27 1.27)
+				)
+				(justify top)
+			)
+		)
+		(property "Value" "100"
+			(at 156.21 83.82 90)
+			(show_name no)
+			(do_not_autoplace no)
+			(effects
+				(font
+					(size 1.27 1.27)
+				)
+			)
+		)
+		(property "Footprint" "Resistor_SMD:R_0402_1005Metric"
+			(at 154.432 83.82 90)
+			(hide yes)
+			(show_name no)
+			(do_not_autoplace no)
+			(effects
+				(font
+					(size 1.27 1.27)
+				)
+			)
+		)
+		(property "Datasheet" ""
+			(at 156.21 83.82 0)
+			(hide yes)
+			(show_name no)
+			(do_not_autoplace no)
+			(effects
+				(font
+					(size 1.27 1.27)
+				)
+			)
+		)
+		(property "Description" "Resistor"
+			(at 156.21 83.82 0)
+			(hide yes)
+			(show_name no)
+			(do_not_autoplace no)
+			(effects
+				(font
+					(size 1.27 1.27)
+				)
+			)
+		)
+		(property "LCSC" "C25076"
+			(at 156.21 83.82 90)
+			(hide yes)
+			(show_name no)
+			(do_not_autoplace no)
+			(effects
+				(font
+					(size 1.27 1.27)
+				)
+			)
+		)
+		(property "Stock" "Basic"
+			(at 156.21 83.82 90)
+			(hide yes)
+			(show_name no)
+			(do_not_autoplace no)
+			(effects
+				(font
+					(size 1.27 1.27)
+				)
+			)
+		)
+		(pin "2"
+		)
+		(pin "1"
+		)
+		(instances
+			(project "gpsfreak"
+				(path "/3160ff17-81c2-4674-af97-e8d9acaf6b65/4b25ac19-17bc-44e9-ba12-1d7cffc23283"
+					(reference "R65")
+					(unit 1)
+				)

Commit message: Change the 10µF 0402 part number.
Parts:
- C81, C85: LCSC C15525 -> C315248; Stock Basic -> Ext
Changed lines of the file:
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@@
 		)
 		(property "Intersheetrefs" "${INTERSHEET_REFS}"
-			(at 97.4658 82.55 0)
+			(at 96.4498 82.55 0)
 			(show_name no)
 			(do_not_autoplace no)
@@
 			)
 		)
-		(property "Datasheet" ""
+		(property "Datasheet" "10V"
 			(at 173.99 67.31 0)
 			(hide yes)
@@
 			)
 		)
-		(property "LCSC" "C15525"
+		(property "LCSC" "C315248"
 			(at 173.99 67.31 0)
 			(hide yes)
@@
 			)
 		)
-		(property "Stock" "Basic"
+		(property "Stock" "Ext"
 			(at 173.99 67.31 0)
 			(hide yes)
@@
 			)
 		)
-		(property "Datasheet" ""
+		(property "Datasheet" "10V"
 			(at 194.31 67.31 0)
 			(hide yes)
@@
 			)
 		)
-		(property "LCSC" "C15525"
+		(property "LCSC" "C315248"
 			(at 194.31 67.31 0)
 			(hide yes)
@@
 			)
 		)
-		(property "Stock" "Basic"
+		(property "Stock" "Ext"
 			(at 194.31 67.31 0)
 			(hide yes)
